File: kicad/colored_noise_generator.kicad_sch (KiCad schematic)
At the start: 43 parts, among them J2 Screw_Terminal_01x03, J3 Conn_01x03, J4 Conn_01x02, Q1 2N2905A, SW1 DPDT, SW2 DP3T, U1 LT1013CP, U2 LT1013CP

Commit message: Change component values while referring to simulation results
Parts:
- C4, C9: value 10u -> 1u
- R13, R18, R20: value 22k -> 220k
- R2: value 100k -> 10k
- R21: value 1Meg -> 820k
- R24: value 22k -> 180k
Other:
- note added: "2*pi*C1*R2 => 1.59 Hz"
- note added: "2*pi*C4*R13 = 2*pi*C10*R18 => 0.723 Hz"
- note added: "2*pi*C4*R20 => fc_min = 0.723 Hz 2*pi*C8*R23 => fc_max = 18.55 Hz"
- note added: "2*pi*C5*R15 => 10.8 kHz"
- note added: "2*pi*C6*R16 => 723 Hz"
- note added: "2*pi*C7*R17 => 86.1 Hz"
- note added: "2*pi*C9*RV1 => fc_min = 7.96 Hz"
- note added: "White: |Gain| = R22/R13 Pink: |Gain| = (R14/R18)*(R22/R21) Brown: |Gain| = (R22/R24)*(R23/(R20+R23)) Ratios determined via simulation to get roughly all equal to 13 dB"
- note added: "|Gain| = R3/R2 + 1 = 41 dB"
- note removed: "White: |Gain| = R22/R13 Pink: |Gain| = (R14/R18)*(R22/R21) Brown: |Gain| = R22/R24 All equal: = 33 dB"
- note removed: "fc = 2*pi*C1*R2 = 1.59 Hz"
- note removed: "fc = 2*pi*C4*R13 = 2*pi*C10*R18 = 0.723 Hz"
- note removed: "fc = 2*pi*C5*R15 = 10.8 kHz"
- note removed: "fc = 2*pi*C6*R16 = 723 Hz"
- note removed: "fc = 2*pi*C7*R17 = 86.1 Hz"
- note removed: "fc_min = 2*pi*C14*R20 = 0.723 Hz fc_max = 2*pi*C8*R23 = 18.55 Hz"
- note removed: "fc_min = 2*pi*C9*RV1 = 0.796 Hz"
- note removed: "|Gain| = R3/R2 + 1 = 21 dB"
- moved on the sheet: C9, J4, R19, VR1
