File: kicad/sim/colored_noise_generator_sim.kicad_sch (KiCad schematic)
At the start: 49 parts, among them U1 OPAMP, U2 OPAMP, U3 OPAMP, U4 OPAMP, U5 OPAMP, U6 OPAMP, U7 OPAMP, U8 OPAMP

Commit message: Change component values while referring to simulation results
Parts:
- added R24: 820k, symbol Device:R_Small
- added R25: 1Meg, symbol Device:R_Small
- C13, C14, C15, C3, C4, C5, C6, C7, C9: value 10u -> 1u
- C8: value 90n -> 22n
- R10, R8, R9: value 22k -> 220k
- R13: value 22k -> 180k
- R18, R20, R21: value 1k -> 10k
- R2, R4, R6: value 100k -> 1Meg
- R7: value 100k -> 390k
- U1, U2, U3, U4, U5, U6, U7, U8: Spice_Lib_File libraries/ad8051.lib -> ../libraries/ad8051.lib
Connections:
- net GND: now also U8.1 (+)
- net at R12.2, R14.2, R15.2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: now also R24.2; no longer U8.1 (+)
- net at C15.1, U8.3: now also R25.2; no longer U8.2 (-)
- new net: R24.1, R25.1, U8.2 (-)
Other:
- note added: "Brown noise"
- note added: "Pink noise"
- note added: "White noise"
- moved on the sheet: C3, R1, R2
